File: kicad/nobmc.kicad_pcb (KiCad board)
At the start: 2 copper layers, 35 x 20 mm, 18 parts, among them J1 Conn_01x06, Q1 2N7002K, Q2 2N7002K

Commit message: Refresh with Kicad 9.0
Parts:
- HOLE (x2): footprint ToolingHole_1.152mm -> MountingHole:ToolingHole_1.152mm
Routing:
- net /GND: track 13.9 -> 0.00 mm, vias 3 -> 0
- net Net-(D1-K): track 31.9 -> 28.4 mm
- added copper zone on F.Cu, net /GND
Other:
- board text added: "NoBMC 1.1 2026-07-16"
- board text removed: "NoBMC 1.0 2023-02-15"
